Commit message: urdf: make leg joints movable

File: src/robot_description/hexapod.urdf.xacro (robot description, xacro)
@@ -20,5 +20,12 @@
   <!-- legs -->
   <xacro:macro name="leg" params="index reflect xyz rpy">
-    <!-- leg_aX: upper segment (shoulder) -->
+    <!-- leg_X: fixed to base_link -->
+    <link name="leg_${index}" />
+    <joint name="base_link__leg_${index}" type="fixed">
+      <parent link="base_link" />
+      <child link="leg_${index}" />
+      <origin xyz="${xyz}" rpy="${rpy}" />
+    </joint>
+    <!-- leg_Xa: shoulder  -->
     <link name="leg_${index}a">
       <visual>
@@ -29,10 +36,18 @@
       </visual>
     </link>
-    <joint name="base_link__leg_${index}a" type="fixed">
-      <parent link="base_link" />
+    <joint name="leg_${index}_base__leg_${index}a" type="revolute">
+      <axis xyz="0 0 1" />
+      <xacro:if value="${reflect == 1}">
+        <limit lower="${joint_a_limit_lower}" upper="${joint_a_limit_upper}"
+            effort="${joint_effort}" velocity="${joint_velocity}" />
+      </xacro:if>
+      <xacro:unless value="${reflect == 1}">
+        <limit lower="${-joint_a_limit_upper}" upper="${-joint_a_limit_lower}"
+            effort="${joint_effort}" velocity="${joint_velocity}" />
+      </xacro:unless>
+      <parent link="leg_${index}" />
       <child link="leg_${index}a" />
-      <origin xyz="${xyz}" rpy="${rpy}" />
     </joint>
-    <!-- leg_bX: center segment -->
+    <!-- leg_Xb: upper segment -->
     <link name="leg_${index}b">
       <visual>
@@ -43,10 +58,19 @@
       </visual>
     </link>
-    <joint name="base_link__leg_${index}b" type="fixed">
+    <joint name="leg_${index}a__leg_${index}b" type="revolute">
+      <axis xyz="1 0 0" />
+      <xacro:if value="${reflect == 1}">
+        <limit lower="${joint_b_limit_lower}" upper="${joint_b_limit_upper}"
+            effort="${joint_effort}" velocity="${joint_velocity}" />
+      </xacro:if>
+      <xacro:unless value="${reflect == 1}">
+        <limit lower="${-joint_b_limit_upper}" upper="${-joint_b_limit_lower}"
+            effort="${joint_effort}" velocity="${joint_velocity}" />
+      </xacro:unless>
       <parent link="leg_${index}a" />
       <child link="leg_${index}b" />
       <origin xyz="0 ${leg_a_length*reflect} 0" />
     </joint>
-    <!-- leg_cX: lower segment (with foot) -->
+    <!-- leg_Xc: lower segment (with foot) -->
     <link name="leg_${index}c">
       <visual>
@@ -70,5 +94,14 @@
       </collision>
     </link>
-    <joint name="base_link__leg_${index}c" type="fixed">
+    <joint name="leg_${index}b__leg_${index}c" type="revolute">
+      <axis xyz="1 0 0" />
+      <xacro:if value="${reflect == 1}">
+        <limit lower="${joint_c_limit_lower}" upper="${joint_c_limit_upper}"
+            effort="${joint_effort}" velocity="${joint_velocity}" />
+      </xacro:if>
+      <xacro:unless value="${reflect == 1}">
+        <limit lower="${-joint_c_limit_upper}" upper="${-joint_c_limit_lower}"
+            effort="${joint_effort}" velocity="${joint_velocity}" />
+      </xacro:unless>
       <parent link="leg_${index}b" />
       <child link="leg_${index}c" />
@@ -77,7 +110,7 @@
   </xacro:macro>
   <!-- Instantiate the six legs -->
-  <xacro:leg index="0" reflect=" 1" xyz=" 0.15  0.10 0.0" rpy="0 0 -${leg_spreading_angle}" />
-  <xacro:leg index="1" reflect=" 1" xyz=" 0.00  0.15 0.0" rpy="0 0 0" />
-  <xacro:leg index="2" reflect=" 1" xyz="-0.15  0.10 0.0" rpy="0 0 ${leg_spreading_angle}" />
+  <xacro:leg index="0" reflect="1"  xyz=" 0.15  0.10 0.0" rpy="0 0 -${leg_spreading_angle}" />
+  <xacro:leg index="1" reflect="1"  xyz=" 0.00  0.15 0.0" rpy="0 0 0" />
+  <xacro:leg index="2" reflect="1"  xyz="-0.15  0.10 0.0" rpy="0 0 ${leg_spreading_angle}" />
   <xacro:leg index="3" reflect="-1" xyz=" 0.15 -0.10 0.0" rpy="0 0 ${leg_spreading_angle}" />
   <xacro:leg index="4" reflect="-1" xyz=" 0.00 -0.15 0.0" rpy="0 0 0" />

File: src/robot_description/properties.urdf.xacro (robot description, xacro)
@@ -17,3 +17,11 @@
   <xacro:property name="leg_b_length" value="0.150" />
   <xacro:property name="leg_c_length" value="0.150" />
+  <xacro:property name="joint_velocity" value="5.6" />
+  <xacro:property name="joint_effort" value="0.9" />
+  <xacro:property name="joint_a_limit_lower" value="-0.7854" />
+  <xacro:property name="joint_a_limit_upper" value="0.7854" />
+  <xacro:property name="joint_b_limit_lower" value="-1.047" />
+  <xacro:property name="joint_b_limit_upper" value="0.7854" />
+  <xacro:property name="joint_c_limit_lower" value="-2.0944" />
+  <xacro:property name="joint_c_limit_upper" value="0" />
 </robot>

Commit message: urdf: add inertia
and a few other physical parameters

File: src/robot_description/hexapod.urdf.xacro (robot description, xacro)
@@ -17,8 +17,15 @@
       <material name="frame" />
     </visual>
+    <inertial>
+      <mass value="0.600" />
+      <origin xyz="0 0 0" />
+      <inertia ixx="0.0021" iyy="0.0046" izz="0.0065"
+               ixy="0" ixz="0" iyz="0" />
+    </inertial>
   </link>
   <!-- legs -->
   <xacro:macro name="leg" params="index reflect xyz rpy">
     <!-- leg_X: fixed to base_link -->
+    <!-- TODO for Gazebo add inertial if whole link gets ignored -->
     <link name="leg_${index}" />
     <joint name="base_link__leg_${index}" type="fixed">
@@ -35,4 +42,10 @@
         </geometry>
       </visual>
+      <inertial>
+        <mass value="0.100" />
+        <origin xyz="0 ${leg_a_length/2*reflect} 0" />
+        <inertia ixx="0.000028" iyy="0.000028" izz="0.000028"
+                 ixy="0"        ixz="0"        iyz="0" />
+      </inertial>
     </link>
     <joint name="leg_${index}_base__leg_${index}a" type="revolute">
@@ -48,4 +61,5 @@
       <parent link="leg_${index}" />
       <child link="leg_${index}a" />
+      <dynamics friction="${joint_friction}" />
     </joint>
     <!-- leg_Xb: upper segment -->
@@ -57,4 +71,10 @@
         </geometry>
       </visual>
+      <inertial>
+        <mass value="0.100" />
+        <origin xyz="0 ${leg_b_length/2*reflect} 0" />
+        <inertia ixx="0.000195" iyy="0.000010" izz="0.000195"
+                 ixy="0"        ixz="0"        iyz="0" />
+      </inertial>
     </link>
     <joint name="leg_${index}a__leg_${index}b" type="revolute">
@@ -71,4 +91,5 @@
       <child link="leg_${index}b" />
       <origin xyz="0 ${leg_a_length*reflect} 0" />
+      <dynamics friction="${joint_friction}" />
     </joint>
     <!-- leg_Xc: lower segment (with foot) -->
@@ -92,5 +113,12 @@
           <sphere radius="0.03" />
         </geometry>
+        <contact_coefficients mu="0.7" />
       </collision>
+      <inertial>
+        <mass value="0.100" />
+        <origin xyz="0 ${leg_c_length/2*reflect} 0" />
+        <inertia ixx="0.000195" iyy="0.000010" izz="0.000195"
+                 ixy="0"        ixz="0"        iyz="0" />
+      </inertial>
     </link>
     <joint name="leg_${index}b__leg_${index}c" type="revolute">
@@ -107,4 +135,5 @@
       <child link="leg_${index}c" />
       <origin xyz="0 ${leg_b_length*reflect} 0" />
+      <dynamics friction="${joint_friction}" />
     </joint>
   </xacro:macro>

File: src/robot_description/properties.urdf.xacro (robot description, xacro)
@@ -19,4 +19,5 @@
   <xacro:property name="joint_velocity" value="5.6" />
   <xacro:property name="joint_effort" value="0.9" />
+  <xacro:property name="joint_friction" value="0.1" />
   <xacro:property name="joint_a_limit_lower" value="-0.7854" />
   <xacro:property name="joint_a_limit_upper" value="0.7854" />

Commit message: sim: get odometry publisher to work
IMU publisher doesn't work yet

File: src/robot_description/hexapod.urdf.xacro (robot description, xacro)
@@ -145,5 +145,14 @@
   <xacro:leg index="4" reflect="-1" xyz=" 0.00 -0.15 0.0" rpy="0 0 0" />
   <xacro:leg index="5" reflect="-1" xyz="-0.15 -0.10 0.0" rpy="0 0 -${leg_spreading_angle}" />
+  <!-- Sensors -->
+  <link name="imu" />
+  <joint name="base_link__imu" type="fixed">
+    <parent link="base_link" />
+    <child link="imu" />
+    <!-- TODO set correct pose -->
+    <origin xyz="0 0 0.05" />
+  </joint>
   <!-- Gazebo (simulation only) -->
+  <!-- docs: https://github.com/gazebosim/gz-sim/tree/main/src/systems -->
   <gazebo>
     <plugin
@@ -153,5 +162,5 @@
       <odom_topic>/model/hexapod/odometry</odom_topic>
       <odom_frame>world</odom_frame>
-      <robot_base_frame>base_footprint</robot_base_frame>
+      <robot_base_frame>base_link</robot_base_frame>
     </plugin>
     <plugin
@@ -160,13 +169,9 @@
       <topic>/model/hexapod/joint_state</topic>
     </plugin>
-    <!-- TODO check this one -->
-    <!--
+    <!-- TODO doesn't work, no imu topic in Gazebo gets published -->
     <plugin
-      filename="ignition-gazebo-imu-sensor-publisher-system"
-      name="ignition::gazebo::systems::ImuSensorPublisher">
-      <update_rate>50</update_rate>
-      <topic>/model/hexapod/imu</topic>
+      filename="ignition-gazebo-imu-system"
+      name="ignition::gazebo::systems::Imu">
     </plugin>
-    -->
   </gazebo>
 </robot>

Commit message: sim: add servo drives
Add servo drives in the form of JointPositionController instances.
The servo parameters were guessed from the Hiwonder specs
and at first sight the reference tracking is fine -
some overshoot but no oscillations.

The servo drives can be commanded from the command line using e.g.
```
ros2 topic pub /actuators actuator_msgs/msg/Actuators \
"{position: [0.0, 0.0, 0.0, 0.0, 0.0, 0.0, 0.0, 0.0, 0.0, \
0.0, 0.0, 0.0, 0.0, 0.0, 0.0, 0.0, 0.0, 0.0]}"
```

File: src/robot_description/hexapod.urdf.xacro (robot description, xacro)
@@ -17,4 +17,9 @@
       <material name="frame" />
     </visual>
+    <collision>
+      <geometry>
+        <box size="0.300 0.200 0.050" />
+      </geometry>
+    </collision>
     <inertial>
       <mass value="0.600" />
@@ -25,4 +30,20 @@
   </link>
   <!-- legs -->
+  <xacro:macro name="servo" params="index joint_name">
+    <gazebo>
+      <plugin
+        filename="gz-sim-joint-position-controller-system"
+        name="gz::sim::systems::JointPositionController">
+        <joint_name>${joint_name}</joint_name>
+        <use_actuator_msg>true</use_actuator_msg>
+        <actuator_number>${index}</actuator_number>
+        <cmd_max>${servo_effort_limit}</cmd_max>
+        <cmd_min>${-servo_effort_limit}</cmd_min>
+        <p_gain>${servo_p_gain}</p_gain>
+        <i_gain>0.</i_gain>
+        <d_gain>0.</d_gain>
+      </plugin>
+    </gazebo>
+  </xacro:macro>
   <xacro:macro name="leg" params="index reflect xyz rpy">
     <!-- leg_X: fixed to base_link -->
@@ -53,13 +74,13 @@
       <xacro:if value="${reflect == 1}">
         <limit lower="${joint_a_limit_lower}" upper="${joint_a_limit_upper}"
-            effort="${joint_effort}" velocity="${joint_velocity}" />
+            effort="${servo_effort_limit}" velocity="${servo_velocity_limit}" />
       </xacro:if>
       <xacro:unless value="${reflect == 1}">
         <limit lower="${-joint_a_limit_upper}" upper="${-joint_a_limit_lower}"
-            effort="${joint_effort}" velocity="${joint_velocity}" />
+            effort="${servo_effort_limit}" velocity="${servo_velocity_limit}" />
       </xacro:unless>
       <parent link="leg_${index}" />
       <child link="leg_${index}a" />
-      <dynamics friction="${joint_friction}" />
+      <dynamics friction="${servo_static_friction}" damping="${servo_damping_friction}" />
     </joint>
     <!-- leg_Xb: upper segment -->
@@ -82,14 +103,14 @@
       <xacro:if value="${reflect == 1}">
         <limit lower="${joint_b_limit_lower}" upper="${joint_b_limit_upper}"
-            effort="${joint_effort}" velocity="${joint_velocity}" />
+            effort="${servo_effort_limit}" velocity="${servo_velocity_limit}" />
       </xacro:if>
       <xacro:unless value="${reflect == 1}">
         <limit lower="${-joint_b_limit_upper}" upper="${-joint_b_limit_lower}"
-            effort="${joint_effort}" velocity="${joint_velocity}" />
+            effort="${servo_effort_limit}" velocity="${servo_velocity_limit}" />
       </xacro:unless>
       <parent link="leg_${index}a" />
       <child link="leg_${index}b" />
       <origin xyz="0 ${leg_a_length*reflect} 0" />
-      <dynamics friction="${joint_friction}" />
+      <dynamics friction="${servo_static_friction}" damping="${servo_damping_friction}" />
     </joint>
     <!-- leg_Xc: lower segment (with foot) -->
@@ -126,15 +147,18 @@
       <xacro:if value="${reflect == 1}">
         <limit lower="${joint_c_limit_lower}" upper="${joint_c_limit_upper}"
-            effort="${joint_effort}" velocity="${joint_velocity}" />
+            effort="${servo_effort_limit}" velocity="${servo_velocity_limit}" />
       </xacro:if>
       <xacro:unless value="${reflect == 1}">
         <limit lower="${-joint_c_limit_upper}" upper="${-joint_c_limit_lower}"
-            effort="${joint_effort}" velocity="${joint_velocity}" />
+            effort="${servo_effort_limit}" velocity="${servo_velocity_limit}" />
       </xacro:unless>
       <parent link="leg_${index}b" />
       <child link="leg_${index}c" />
       <origin xyz="0 ${leg_b_length*reflect} 0" />
-      <dynamics friction="${joint_friction}" />
-    </joint>
+      <dynamics friction="${servo_static_friction}" damping="${servo_damping_friction}" />
+    </joint>
+    <xacro:servo index="${index*3+0}" joint_name="leg_${index}_base__leg_${index}a" />
+    <xacro:servo index="${index*3+1}" joint_name="leg_${index}a__leg_${index}b" />
+    <xacro:servo index="${index*3+2}" joint_name="leg_${index}b__leg_${index}c" />
   </xacro:macro>
   <!-- Instantiate the six legs -->

File: src/robot_description/properties.urdf.xacro (robot description, xacro)
@@ -17,7 +17,9 @@
   <xacro:property name="leg_b_length" value="0.150" />
   <xacro:property name="leg_c_length" value="0.150" />
-  <xacro:property name="joint_velocity" value="5.6" />
-  <xacro:property name="joint_effort" value="0.9" />
-  <xacro:property name="joint_friction" value="0.1" />
+  <xacro:property name="servo_velocity_limit" value="5.6" />
+  <xacro:property name="servo_effort_limit" value="0.9" />
+  <xacro:property name="servo_static_friction" value="0.3" />
+  <xacro:property name="servo_damping_friction" value="0.1" />
+  <xacro:property name="servo_p_gain" value="8.4" />
   <xacro:property name="joint_a_limit_lower" value="-0.7854" />
   <xacro:property name="joint_a_limit_upper" value="0.7854" />

Commit message: add script to move legs + adjust hardware such that it walks
walks => belly flopping

File: src/robot_description/hexapod.urdf.xacro (robot description, xacro)
@@ -23,5 +23,5 @@
     </collision>
     <inertial>
-      <mass value="0.600" />
+      <mass value="0.300" />
       <origin xyz="0 0 0" />
       <inertia ixx="0.0021" iyy="0.0046" izz="0.0065"

File: src/robot_description/properties.urdf.xacro (robot description, xacro)
@@ -14,9 +14,9 @@
   <!-- ********** -->
   <xacro:property name="leg_spreading_angle" value="0.5236" />
-  <xacro:property name="leg_a_length" value="0.050" />
-  <xacro:property name="leg_b_length" value="0.150" />
-  <xacro:property name="leg_c_length" value="0.150" />
+  <xacro:property name="leg_a_length" value="0.060" />
+  <xacro:property name="leg_b_length" value="0.060" />
+  <xacro:property name="leg_c_length" value="0.060" />
   <xacro:property name="servo_velocity_limit" value="5.6" />
-  <xacro:property name="servo_effort_limit" value="0.9" />
+  <xacro:property name="servo_effort_limit" value="1.5" />
   <xacro:property name="servo_static_friction" value="0.3" />
   <xacro:property name="servo_damping_friction" value="0.1" />

Commit message: urdf: add foot link
to allow easy referring to the foot ball center

File: src/robot_description/hexapod.urdf.xacro (robot description, xacro)
@@ -114,5 +114,5 @@
       <dynamics friction="${servo_static_friction}" damping="${servo_damping_friction}" />
     </joint>
-    <!-- leg_Xc: lower segment (with foot) -->
+    <!-- leg_Xc: lower segment -->
     <link name="leg_${index}c">
       <visual>
@@ -157,4 +157,11 @@
       <origin xyz="0 ${leg_b_length*reflect} 0" />
       <dynamics friction="${servo_static_friction}" damping="${servo_damping_friction}" />
+    </joint>
+    <!-- Link in the foot ball center to easily refer to that point in KDL -->
+    <link name="foot_${index}" />
+    <joint name="leg_${index}c__foot_${index}" type="fixed">
+      <parent link="leg_${index}c" />
+      <child link="foot_${index}" />
+      <origin xyz="0 ${leg_c_length*reflect} 0" />
     </joint>
     <xacro:servo index="${index*3+0}" joint_name="leg_${index}_base__leg_${index}a" />

Commit message: urdf: bugfix + increase joint limit
legs 3 and 5 were swapped

File: src/robot_description/hexapod.urdf.xacro (robot description, xacro)
@@ -173,7 +173,7 @@
   <xacro:leg index="1" reflect="1"  xyz=" 0.00  0.15 0.0" rpy="0 0 0" />
   <xacro:leg index="2" reflect="1"  xyz="-0.15  0.10 0.0" rpy="0 0 ${leg_spreading_angle}" />
-  <xacro:leg index="3" reflect="-1" xyz=" 0.15 -0.10 0.0" rpy="0 0 ${leg_spreading_angle}" />
+  <xacro:leg index="3" reflect="-1" xyz="-0.15 -0.10 0.0" rpy="0 0 -${leg_spreading_angle}" />
   <xacro:leg index="4" reflect="-1" xyz=" 0.00 -0.15 0.0" rpy="0 0 0" />
-  <xacro:leg index="5" reflect="-1" xyz="-0.15 -0.10 0.0" rpy="0 0 -${leg_spreading_angle}" />
+  <xacro:leg index="5" reflect="-1" xyz=" 0.15 -0.10 0.0" rpy="0 0 ${leg_spreading_angle}" />
   <!-- Sensors -->
   <link name="imu" />

File: src/robot_description/properties.urdf.xacro (robot description, xacro)
@@ -26,5 +26,5 @@
   <xacro:property name="joint_b_limit_lower" value="-1.047" />
   <xacro:property name="joint_b_limit_upper" value="0.7854" />
-  <xacro:property name="joint_c_limit_lower" value="-2.0944" />
+  <xacro:property name="joint_c_limit_lower" value="-2.618" />
   <xacro:property name="joint_c_limit_upper" value="0" />
 </robot>
