Commit message: urdf: increase servo gain
This should be a more reasonable value, otherwise the tracking error is too large.

File: src/robot_description/properties.urdf.xacro (robot description, xacro)
@@ -21,5 +21,5 @@
   <xacro:property name="servo_static_friction" value="0.3" />
   <xacro:property name="servo_damping_friction" value="0.1" />
-  <xacro:property name="servo_p_gain" value="8.4" />
+  <xacro:property name="servo_p_gain" value="17.8" />
   <xacro:property name="joint_a_limit_lower" value="-0.7854" />
   <xacro:property name="joint_a_limit_upper" value="0.7854" />

Commit message: walking: follow cmd_vel + add timeout + improve motion

File: src/robot_description/properties.urdf.xacro (robot description, xacro)
@@ -16,5 +16,5 @@
   <xacro:property name="leg_a_length" value="0.060" />
   <xacro:property name="leg_b_length" value="0.060" />
-  <xacro:property name="leg_c_length" value="0.060" />
+  <xacro:property name="leg_c_length" value="0.080" />
   <xacro:property name="servo_velocity_limit" value="5.6" />
   <xacro:property name="servo_effort_limit" value="1.5" />

Commit message: tuning: increase speeds and joint limits
Hexapod handles it well, at least in simulation.

File: src/robot_description/properties.urdf.xacro (robot description, xacro)
@@ -25,5 +25,5 @@
   <xacro:property name="joint_a_limit_upper" value="0.7854" />
   <xacro:property name="joint_b_limit_lower" value="-1.047" />
-  <xacro:property name="joint_b_limit_upper" value="0.7854" />
+  <xacro:property name="joint_b_limit_upper" value="1.047" />
   <xacro:property name="joint_c_limit_lower" value="-2.618" />
   <xacro:property name="joint_c_limit_upper" value="0" />
